File: crates/hauksbee-engine/tests/fixtures/verdict_medium_lint.kicad_pcb (KiCad board)
At the start: 4 parts, among them Q1 2N7002

Commit message: Block the ordering verdict on a layout with no copper routing
A .kicad_pcb with placed pads and no routing at all was one Low note, so a
fully modelled but unrouted board could still read OK TO ORDER. It is now one
High unrouted_pad finding saying the board is not routed yet and cannot be
ordered as is. The circuit checks still run on its netlist; the finding gates
through the shared Failing cause, so CLI, --json, CI and the web report give
the same reason line.

Tests that meant something else and only happened to use an unrouted board
now route it: the medium-lint verdict fixture, the waiver-gate boot_gate copy
and I2C lint board, the phantom-short pass case, and QC scenario 10 (a patch
step). The boot_gate web golden and its reason count now include the unrouted
finding, since that board really is unrouted.
Routing:
- net GND: track 0.00 -> 60.0 mm
- net LOAD_DRAIN: track 0.00 -> 31.0 mm
- net +5V: track 0.00 -> 20.0 mm
- net GATE_CTRL: track 0.00 -> 15.0 mm
Changed lines of the file:
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@@
     (pad 2 thru_hole circle (at 2 0) (net 1 "GND"))
   )
+  (segment (start 110 100) (end 110 115) (width 0.25) (layer F.Cu) (net 3))
+  (segment (start 112 100) (end 112 115) (width 0.25) (layer F.Cu) (net 1))
+  (segment (start 112 115) (end 142 115) (width 0.25) (layer F.Cu) (net 1))
+  (segment (start 142 115) (end 142 100) (width 0.25) (layer F.Cu) (net 1))
+  (segment (start 111 100) (end 111 95) (width 0.25) (layer F.Cu) (net 4))
+  (segment (start 111 95) (end 132 95) (width 0.25) (layer F.Cu) (net 4))
+  (segment (start 132 95) (end 132 100) (width 0.25) (layer F.Cu) (net 4))
+  (segment (start 130 100) (end 130 105) (width 0.25) (layer F.Cu) (net 2))
+  (segment (start 130 105) (end 140 105) (width 0.25) (layer F.Cu) (net 2))
+  (segment (start 140 105) (end 140 100) (width 0.25) (layer F.Cu) (net 2))
 )
