File: crates/hauksbee-engine/tests/fixtures/boot_gate_pulldown.kicad_pcb (KiCad board)
At the start: 4 parts, among them Q1 2N7002, U1 ATmega328P

Commit message: Add an MCP1702-3302 SOT-23A card and name the DIP-28 package in ATmega328P fixtures
Parts:
- U1: footprint Package_QFP:TQFP-32_7x7mm_P0.8mm -> Package_DIP:DIP-28_W7.62mm
Changed lines of the file:
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@@
   (net 3 "GATE_CTRL")
   (net 4 "LOAD_DRAIN")
-  (module Package_QFP:TQFP-32_7x7mm_P0.8mm (layer F.Cu)
+  (module Package_DIP:DIP-28_W7.62mm (layer F.Cu)
     (at 100 100)
     (fp_text reference U1 (at 0 0) (layer F.SilkS))
