File: frontend/public/samples/boot_gate.kicad_pcb (KiCad board)
At the start: 2 copper layers, 3 parts, among them Q1 2N7002, U1 ATmega328P

Commit message: Add an MCP1702-3302 SOT-23A card and name the DIP-28 package in ATmega328P fixtures
Parts:
- U1: footprint Package_QFP:TQFP-32_7x7mm_P0.8mm -> Package_DIP:DIP-28_W7.62mm
Changed lines of the file:
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@@
-(kicad_pcb(version 20171130)(generator "pcbnew")(general(thickness 1.6))(paper "A4")(layers(0 "F.Cu"signal)(31 "B.Cu"signal)(36 "B.SilkS"user)(37 "F.SilkS"user)(38 "B.Mask"user)(39 "F.Mask"user)(44 "Edge.Cuts"user)(48 "B.Fab"user)(49 "F.Fab"user))(setup(pad_to_mask_clearance 0))(net 0 "")(net 1 "+5V")(net 2 "GND")(net 3 "GATE_CTRL")(net 4 "LOAD_DRAIN")(footprint "Package_TO_SOT_SMD:SOT-23"(layer "F.Cu")(at 4.974 0.902 0)(property "Reference""Q1")(property "Value""2N7002")(pad G smd rect(at 0 0 0)(size 0.6 0.6)(layers "F.Cu")(net 3 "GATE_CTRL"))(pad D smd rect(at 1 0 0)(size 0.6 0.6)(layers "F.Cu")(net 4 "LOAD_DRAIN"))(pad S smd rect(at 2 0 0)(size 0.6 0.6)(layers "F.Cu")(net 2 "GND")))(footprint "Package_QFP:TQFP-32_7x7mm_P0.8mm"(layer "F.Cu")(at -4.073 3.415 0)(property "Reference""U1")(property "Value""ATmega328P")(pad 7 smd rect(at -3 0 0)(size 0.6 0.6)(layers "F.Cu")(net 1 "+5V"))(pad 8 smd rect(at -3 1 0)(size 0.6 0.6)(layers "F.Cu")(net 2 "GND"))(pad 14 smd rect(at 3 0 0)(size 0.6 0.6)(layers "F.Cu")(net 3 "GATE_CTRL"))(pad 20 smd rect(at 3 1 0)(size 0.6 0.6)(layers "F.Cu")(net 1 "+5V"))(pad 22 smd rect(at 3 2 0)(size 0.6 0.6)(layers "F.Cu")(net 2 "GND")))(footprint "Resistor_THT:R_Axial_DIN0207_L6.3mm_D2.5mm"(layer "F.Cu")(at 0.032 -5.231 0)(property "Reference""R1")(property "Value""1k")(pad 1 thru_hole circle(at 0 0 0)(size 0.6 0.6)(layers "F.Cu")(net 1 "+5V"))(pad 2 thru_hole circle(at 2 0 0)(size 0.6 0.6)(layers "F.Cu")(net 4 "LOAD_DRAIN")))(segment(start -1.073 4.415)(end -4.67 4.415)(width 0.25)(layer "F.Cu")(net 1))(segment(start -4.67 4.415)(end -5.67 3.415)(width 0.25)(layer "F.Cu")(net 1))(segment(start -5.67 3.415)(end -7.073 3.415)(width 0.25)(layer "F.Cu")(net 1))(segment(start 0.032 -5.231)(end -7.073 1.874)(width 0.25)(layer "F.Cu")(net 1))(segment(start -7.073 1.874)(end -7.073 3.415)(width 0.25)(layer "F.Cu")(net 1))(segment(start -1.073 3.415)(end 1.63583 3.415)(width 0.25)(layer "F.Cu")(net 3))(segment(start 1.63583 3.415)(end 4.14883 0.902)(width 0.25)(layer "F.Cu")(net 3))(segment(start 4.974 0.902)(end 4.14883 0.902)(width 0.25)(layer "F.Cu")(net 3))(segment(start -1.073 5.415)(end 3.28617 5.415)(width 0.25)(layer "F.Cu")(net 2))(segment(start 3.28617 5.415)(end 6.974 1.72717)(width 0.25)(layer "F.Cu")(net 2))(segment(start -6.24783 4.415)(end -5.24783 5.415)(width 0.25)(layer "F.Cu")(net 2))(segment(start -5.24783 5.415)(end -1.073 5.415)(width 0.25)(layer "F.Cu")(net 2))(segment(start 6.974 0.902)(end 6.974 1.72717)(width 0.25)(layer "F.Cu")(net 2))(segment(start -7.073 4.415)(end -6.24783 4.415)(width 0.25)(layer "F.Cu")(net 2))(segment(start 2.032 -5.231)(end 5.974 -1.289)(width 0.25)(layer "F.Cu")(net 4))(segment(start 5.974 -1.289)(end 5.974 0.902)(width 0.25)(layer "F.Cu")(net 4)))
+(kicad_pcb(version 20171130)(generator "pcbnew")(general(thickness 1.6))(paper "A4")(layers(0 "F.Cu"signal)(31 "B.Cu"signal)(36 "B.SilkS"user)(37 "F.SilkS"user)(38 "B.Mask"user)(39 "F.Mask"user)(44 "Edge.Cuts"user)(48 "B.Fab"user)(49 "F.Fab"user))(setup(pad_to_mask_clearance 0))(net 0 "")(net 1 "+5V")(net 2 "GND")(net 3 "GATE_CTRL")(net 4 "LOAD_DRAIN")(footprint "Package_TO_SOT_SMD:SOT-23"(layer "F.Cu")(at 4.974 0.902 0)(property "Reference""Q1")(property "Value""2N7002")(pad G smd rect(at 0 0 0)(size 0.6 0.6)(layers "F.Cu")(net 3 "GATE_CTRL"))(pad D smd rect(at 1 0 0)(size 0.6 0.6)(layers "F.Cu")(net 4 "LOAD_DRAIN"))(pad S smd rect(at 2 0 0)(size 0.6 0.6)(layers "F.Cu")(net 2 "GND")))(footprint "Package_DIP:DIP-28_W7.62mm"(layer "F.Cu")(at -4.073 3.415 0)(property "Reference""U1")(property "Value""ATmega328P")(pad 7 smd rect(at -3 0 0)(size 0.6 0.6)(layers "F.Cu")(net 1 "+5V"))(pad 8 smd rect(at -3 1 0)(size 0.6 0.6)(layers "F.Cu")(net 2 "GND"))(pad 14 smd rect(at 3 0 0)(size 0.6 0.6)(layers "F.Cu")(net 3 "GATE_CTRL"))(pad 20 smd rect(at 3 1 0)(size 0.6 0.6)(layers "F.Cu")(net 1 "+5V"))(pad 22 smd rect(at 3 2 0)(size 0.6 0.6)(layers "F.Cu")(net 2 "GND")))(footprint "Resistor_THT:R_Axial_DIN0207_L6.3mm_D2.5mm"(layer "F.Cu")(at 0.032 -5.231 0)(property "Reference""R1")(property "Value""1k")(pad 1 thru_hole circle(at 0 0 0)(size 0.6 0.6)(layers "F.Cu")(net 1 "+5V"))(pad 2 thru_hole circle(at 2 0 0)(size 0.6 0.6)(layers "F.Cu")(net 4 "LOAD_DRAIN")))(segment(start -1.073 4.415)(end -4.67 4.415)(width 0.25)(layer "F.Cu")(net 1))(segment(start -4.67 4.415)(end -5.67 3.415)(width 0.25)(layer "F.Cu")(net 1))(segment(start -5.67 3.415)(end -7.073 3.415)(width 0.25)(layer "F.Cu")(net 1))(segment(start 0.032 -5.231)(end -7.073 1.874)(width 0.25)(layer "F.Cu")(net 1))(segment(start -7.073 1.874)(end -7.073 3.415)(width 0.25)(layer "F.Cu")(net 1))(segment(start -1.073 3.415)(end 1.63583 3.415)(width 0.25)(layer "F.Cu")(net 3))(segment(start 1.63583 3.415)(end 4.14883 0.902)(width 0.25)(layer "F.Cu")(net 3))(segment(start 4.974 0.902)(end 4.14883 0.902)(width 0.25)(layer "F.Cu")(net 3))(segment(start -1.073 5.415)(end 3.28617 5.415)(width 0.25)(layer "F.Cu")(net 2))(segment(start 3.28617 5.415)(end 6.974 1.72717)(width 0.25)(layer "F.Cu")(net 2))(segment(start -6.24783 4.415)(end -5.24783 5.415)(width 0.25)(layer "F.Cu")(net 2))(segment(start -5.24783 5.415)(end -1.073 5.415)(width 0.25)(layer "F.Cu")(net 2))(segment(start 6.974 0.902)(end 6.974 1.72717)(width 0.25)(layer "F.Cu")(net 2))(segment(start -7.073 4.415)(end -6.24783 4.415)(width 0.25)(layer "F.Cu")(net 2))(segment(start 2.032 -5.231)(end 5.974 -1.289)(width 0.25)(layer "F.Cu")(net 4))(segment(start 5.974 -1.289)(end 5.974 0.902)(width 0.25)(layer "F.Cu")(net 4)))
