File: testdata/boards/ultrasonic_cane/ultrasonic_cane.kicad_pcb (KiCad board)
At the start: 2 copper layers, 60 x 44 mm, 29 parts, among them J2 HC-SR04, J3 USB_Micro-B, M1 Vibration_Motor_3V, Q1 AO3400A, SW1 SW_Push, SW2 SW_Push, U1 ATmega328P, U2 AMS1117-3.3, U3 TP4056, U4 BMA423

Commit message: Add an MCP1702-3302 SOT-23A card and name the DIP-28 package in ATmega328P fixtures
Parts:
- U1: footprint Package_QFP:TQFP-32_7x7mm_P0.8mm -> Package_DIP:DIP-28_W7.62mm
Changed lines of the file:
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@@
     (pad "3" smd roundrect (at 0 -1) (size 0.6 1.0) (layers "F.Cu" "F.Paste" "F.Mask") (net 6 "MOTOR_N"))
   )
-  (footprint "Package_QFP:TQFP-32_7x7mm_P0.8mm" (layer "F.Cu") (at 30 20 0) (attr smd)
+  (footprint "Package_DIP:DIP-28_W7.62mm" (layer "F.Cu") (at 30 20 0) (attr smd)
     (property "Reference" "U1" (at 0 -2 0) (layer "F.SilkS"))
     (property "Value" "ATmega328P" (at 0 2 0) (layer "F.Fab"))
