File: crates/hauksbee-ci/tests/fixtures/lm339_vicr_pair_high.kicad_pcb (KiCad board)
At the start: 2 copper layers, 7 parts, among them U1 LM339B

Commit message: Cards: load-switch enable and capacitor fields, motor-driver supply caps, open-drain audit, bootloader RX idle level; UART header names; generic crystal CL
- Load switches (TPS22916/18/19, AP2281, AP2553, AP22815/22615A): EN role/active level, open-EN behaviour (en_open incl. undefined) and required input/output capacitors; regulator_enable, control_held_off and the required-capacitor check consume them.
- Motor drivers (DRV8833, DRV8825, A4988, TB6612FNG): required supply-pin bulk capacitance from the datasheets.
- Open-drain audit: datasheet-stated open-drain interrupt/alert/ready/fault pins marked in pin_capability.open_drain; open_drain_pullup counts a rail with a chip supply pin on it and leaves pads pin_bias already judges.
- MCU ROM-bootloader UART RX: pin_bias rows (opposed_only) on STM32 and ESP32 cards citing AN2606/AN3155 and the reference manuals.
- debug_header: 6-pin FTDI and 4-pin USB-serial headers recognised by their own pin names.
- Crystal: a card-less crystal takes CL from its value; unknown CL abstains with a note.
- lm339 fixtures: reference RPULLUP renamed R5 (RP is a resistor-network designator).

Signed-off-by: ETM-Code <158038827+ETM-Code@users.noreply.github.com>
Parts:
- removed RPULLUP: 10k, Resistor_SMD:R_0805_2012Metric
- added R5: 10k, Resistor_SMD:R_0805_2012Metric, B.Cu at (160.0, 20.0)
Changed lines of the file:
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@@
-(kicad_pcb(version 1)(generator "pcbnew")(general(thickness 1.6))(paper "A4")(layers(0 "F.Cu"signal)(31 "B.Cu"signal)(36 "B.SilkS"user)(37 "F.SilkS"user)(38 "B.Mask"user)(39 "F.Mask"user)(44 "Edge.Cuts"user)(48 "B.Fab"user)(49 "F.Fab"user))(setup(pad_to_mask_clearance 0))(net 0 "")(net 1 "OUT")(net 2 "V5")(net 3 "INM")(net 4 "INP")(net 5 "GND")(footprint "Package_DIP:DIP-14_W7.62mm"(layer "F.Cu")(at 10 20 0)(property "Reference""U1")(property "Value""LM339B")(pad 1 thru_hole circle(at 2.54 0 0)(size 1.7 1.7)(drill 1)(layers "F.Cu""B.Cu"))(pad 2 thru_hole circle(at 5.08 0 0)(size 1.7 1.7)(drill 1)(layers "F.Cu""B.Cu")(net 1 "OUT"))(pad 3 thru_hole circle(at 7.62 0 0)(size 1.7 1.7)(drill 1)(layers "F.Cu""B.Cu")(net 2 "V5"))(pad 4 thru_hole circle(at 10.16 0 0)(size 1.7 1.7)(drill 1)(layers "F.Cu""B.Cu")(net 3 "INM"))(pad 5 thru_hole circle(at 12.7 0 0)(size 1.7 1.7)(drill 1)(layers "F.Cu""B.Cu")(net 4 "INP"))(pad 6 thru_hole circle(at 15.24 0 0)(size 1.7 1.7)(drill 1)(layers "F.Cu""B.Cu")(net 5 "GND"))(pad 7 thru_hole circle(at 17.78 0 0)(size 1.7 1.7)(drill 1)(layers "F.Cu""B.Cu")(net 5 "GND"))(pad 8 thru_hole circle(at 20.32 0 0)(size 1.7 1.7)(drill 1)(layers "F.Cu""B.Cu")(net 5 "GND"))(pad 9 thru_hole circle(at 22.86 0 0)(size 1.7 1.7)(drill 1)(layers "F.Cu""B.Cu")(net 5 "GND"))(pad 10 thru_hole circle(at 25.4 0 0)(size 1.7 1.7)(drill 1)(layers "F.Cu""B.Cu")(net 5 "GND"))(pad 11 thru_hole circle(at 27.94 0 0)(size 1.7 1.7)(drill 1)(layers "F.Cu""B.Cu")(net 5 "GND"))(pad 12 thru_hole circle(at 30.48 0 0)(size 1.7 1.7)(drill 1)(layers "F.Cu""B.Cu")(net 5 "GND"))(pad 13 thru_hole circle(at 33.02 0 0)(size 1.7 1.7)(drill 1)(layers "F.Cu""B.Cu"))(pad 14 thru_hole circle(at 35.56 0 0)(size 1.7 1.7)(drill 1)(layers "F.Cu""B.Cu")))(footprint "Resistor_SMD:R_0805_2012Metric"(layer "F.Cu")(at 40 20 0)(property "Reference""R1")(property "Value""10k")(pad 1 thru_hole circle(at 2.54 0 0)(size 1.7 1.7)(drill 1)(layers "F.Cu""B.Cu")(net 2 "V5"))(pad 2 thru_hole circle(at 5.08 0 0)(size 1.7 1.7)(drill 1)(layers "F.Cu""B.Cu")(net 4 "INP")))(footprint "Resistor_SMD:R_0805_2012Metric"(layer "F.Cu")(at 70 20 0)(property "Reference""R2")(property "Value""62k")(pad 1 thru_hole circle(at 2.54 0 0)(size 1.7 1.7)(drill 1)(layers "F.Cu""B.Cu")(net 4 "INP"))(pad 2 thru_hole circle(at 5.08 0 0)(size 1.7 1.7)(drill 1)(layers "F.Cu""B.Cu")(net 5 "GND")))(footprint "Resistor_SMD:R_0805_2012Metric"(layer "F.Cu")(at 100 20 0)(property "Reference""R3")(property "Value""10k")(pad 1 thru_hole circle(at 2.54 0 0)(size 1.7 1.7)(drill 1)(layers "F.Cu""B.Cu")(net 2 "V5"))(pad 2 thru_hole circle(at 5.08 0 0)(size 1.7 1.7)(drill 1)(layers "F.Cu""B.Cu")(net 3 "INM")))(footprint "Resistor_SMD:R_0805_2012Metric"(layer "F.Cu")(at 130 20 0)(property "Reference""R4")(property "Value""40k")(pad 1 thru_hole circle(at 2.54 0 0)(size 1.7 1.7)(drill 1)(layers "F.Cu""B.Cu")(net 3 "INM"))(pad 2 thru_hole circle(at 5.08 0 0)(size 1.7 1.7)(drill 1)(layers "F.Cu""B.Cu")(net 5 "GND")))(footprint "Resistor_SMD:R_0805_2012Metric"(layer "F.Cu")(at 160 20 0)(property "Reference""RPULLUP")(property "Value""10k")(pad 1 thru_hole circle(at 2.54 0 0)(size 1.7 1.7)(drill 1)(layers "F.Cu""B.Cu")(net 1 "OUT"))(pad 2 thru_hole circle(at 5.08 0 0)(size 1.7 1.7)(drill 1)(layers "F.Cu""B.Cu")(net 2 "V5")))(footprint "Capacitor_SMD:C_0805_2012Metric"(layer "F.Cu")(at 190 20 0)(property "Reference""CBYP")(property "Value""100nF")(pad 1 thru_hole circle(at 2.54 0 0)(size 1.7 1.7)(drill 1)(layers "F.Cu""B.Cu")(net 2 "V5"))(pad 2 thru_hole circle(at 5.08 0 0)(size 1.7 1.7)(drill 1)(layers "F.Cu""B.Cu")(net 5 "GND"))))
+(kicad_pcb(version 1)(generator "pcbnew")(general(thickness 1.6))(paper "A4")(layers(0 "F.Cu"signal)(31 "B.Cu"signal)(36 "B.SilkS"user)(37 "F.SilkS"user)(38 "B.Mask"user)(39 "F.Mask"user)(44 "Edge.Cuts"user)(48 "B.Fab"user)(49 "F.Fab"user))(setup(pad_to_mask_clearance 0))(net 0 "")(net 1 "OUT")(net 2 "V5")(net 3 "INM")(net 4 "INP")(net 5 "GND")(footprint "Package_DIP:DIP-14_W7.62mm"(layer "F.Cu")(at 10 20 0)(property "Reference""U1")(property "Value""LM339B")(pad 1 thru_hole circle(at 2.54 0 0)(size 1.7 1.7)(drill 1)(layers "F.Cu""B.Cu"))(pad 2 thru_hole circle(at 5.08 0 0)(size 1.7 1.7)(drill 1)(layers "F.Cu""B.Cu")(net 1 "OUT"))(pad 3 thru_hole circle(at 7.62 0 0)(size 1.7 1.7)(drill 1)(layers "F.Cu""B.Cu")(net 2 "V5"))(pad 4 thru_hole circle(at 10.16 0 0)(size 1.7 1.7)(drill 1)(layers "F.Cu""B.Cu")(net 3 "INM"))(pad 5 thru_hole circle(at 12.7 0 0)(size 1.7 1.7)(drill 1)(layers "F.Cu""B.Cu")(net 4 "INP"))(pad 6 thru_hole circle(at 15.24 0 0)(size 1.7 1.7)(drill 1)(layers "F.Cu""B.Cu")(net 5 "GND"))(pad 7 thru_hole circle(at 17.78 0 0)(size 1.7 1.7)(drill 1)(layers "F.Cu""B.Cu")(net 5 "GND"))(pad 8 thru_hole circle(at 20.32 0 0)(size 1.7 1.7)(drill 1)(layers "F.Cu""B.Cu")(net 5 "GND"))(pad 9 thru_hole circle(at 22.86 0 0)(size 1.7 1.7)(drill 1)(layers "F.Cu""B.Cu")(net 5 "GND"))(pad 10 thru_hole circle(at 25.4 0 0)(size 1.7 1.7)(drill 1)(layers "F.Cu""B.Cu")(net 5 "GND"))(pad 11 thru_hole circle(at 27.94 0 0)(size 1.7 1.7)(drill 1)(layers "F.Cu""B.Cu")(net 5 "GND"))(pad 12 thru_hole circle(at 30.48 0 0)(size 1.7 1.7)(drill 1)(layers "F.Cu""B.Cu")(net 5 "GND"))(pad 13 thru_hole circle(at 33.02 0 0)(size 1.7 1.7)(drill 1)(layers "F.Cu""B.Cu"))(pad 14 thru_hole circle(at 35.56 0 0)(size 1.7 1.7)(drill 1)(layers "F.Cu""B.Cu")))(footprint "Resistor_SMD:R_0805_2012Metric"(layer "F.Cu")(at 40 20 0)(property "Reference""R1")(property "Value""10k")(pad 1 thru_hole circle(at 2.54 0 0)(size 1.7 1.7)(drill 1)(layers "F.Cu""B.Cu")(net 2 "V5"))(pad 2 thru_hole circle(at 5.08 0 0)(size 1.7 1.7)(drill 1)(layers "F.Cu""B.Cu")(net 4 "INP")))(footprint "Resistor_SMD:R_0805_2012Metric"(layer "F.Cu")(at 70 20 0)(property "Reference""R2")(property "Value""62k")(pad 1 thru_hole circle(at 2.54 0 0)(size 1.7 1.7)(drill 1)(layers "F.Cu""B.Cu")(net 4 "INP"))(pad 2 thru_hole circle(at 5.08 0 0)(size 1.7 1.7)(drill 1)(layers "F.Cu""B.Cu")(net 5 "GND")))(footprint "Resistor_SMD:R_0805_2012Metric"(layer "F.Cu")(at 100 20 0)(property "Reference""R3")(property "Value""10k")(pad 1 thru_hole circle(at 2.54 0 0)(size 1.7 1.7)(drill 1)(layers "F.Cu""B.Cu")(net 2 "V5"))(pad 2 thru_hole circle(at 5.08 0 0)(size 1.7 1.7)(drill 1)(layers "F.Cu""B.Cu")(net 3 "INM")))(footprint "Resistor_SMD:R_0805_2012Metric"(layer "F.Cu")(at 130 20 0)(property "Reference""R4")(property "Value""40k")(pad 1 thru_hole circle(at 2.54 0 0)(size 1.7 1.7)(drill 1)(layers "F.Cu""B.Cu")(net 3 "INM"))(pad 2 thru_hole circle(at 5.08 0 0)(size 1.7 1.7)(drill 1)(layers "F.Cu""B.Cu")(net 5 "GND")))(footprint "Resistor_SMD:R_0805_2012Metric"(layer "F.Cu")(at 160 20 0)(property "Reference""R5")(property "Value""10k")(pad 1 thru_hole circle(at 2.54 0 0)(size 1.7 1.7)(drill 1)(layers "F.Cu""B.Cu")(net 1 "OUT"))(pad 2 thru_hole circle(at 5.08 0 0)(size 1.7 1.7)(drill 1)(layers "F.Cu""B.Cu")(net 2 "V5")))(footprint "Capacitor_SMD:C_0805_2012Metric"(layer "F.Cu")(at 190 20 0)(property "Reference""CBYP")(property "Value""100nF")(pad 1 thru_hole circle(at 2.54 0 0)(size 1.7 1.7)(drill 1)(layers "F.Cu""B.Cu")(net 2 "V5"))(pad 2 thru_hole circle(at 5.08 0 0)(size 1.7 1.7)(drill 1)(layers "F.Cu""B.Cu")(net 5 "GND"))))
